File: schematic/coleco_original.kicad_sch (KiCad schematic)
At the start: 0 parts

Commit message: added u5 decoder lines, need to rename for chip selects that they actually are in future.
Other:
- sheet clock_reset ports: added E2_U6, RFSH; removed E2
- sheet decoder_logic ports: added E2_U6, E3_U5, RFSH, U5_O1, U5_O2, U5_O3, U5_O4, U5_O5, U5_O6, U5_O7; removed E2
- sheet io_ports ports: added E3_U5, U5_O1, U5_O2, U5_O4, U5_O5, U5_O6, U5_O7; removed none
- sheet storage ports: added U5_O3; removed none

Commit message: added u6 decoder lines, renamed a few lines to make sense to there destination.
Other:
- sheet controller ports: added U6_O0, U6_O4, U6_O7; removed none
- sheet decoder_logic ports: added U6_O0, U6_O4, U6_O7, ~{CSR}, ~{CSW}, ~{RAM_CS}, ~{ROM_ENABLE}, ~{SND_ENABLE}; removed U5_O0, U5_O3
- sheet sound ports: added ~{SND_ENABLE}; removed none
- sheet storage ports: added ~{RAM_CS}, ~{ROM_ENABLE}; removed U5_O0, U5_O3
- sheet video ports: added ~{CSR}, ~{CSW}; removed none
