File: schematic/cpu.kicad_sch (KiCad schematic)
At the start: 3 parts, among them U1 Z80CPU

Commit message: added pdf schematic, cleanup pdf files, added 3D image, updated readme
Other:
- title: Reverse Engineer Colecovision -> Righteous Tentacle, Colecovision Reverse Engineering Project
Changed lines of the file:
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@@
   (paper "USLetter")
   (title_block
-    (title "Reverse Engineer Colecovision")
+    (title "Righteous Tentacle, Colecovision Reverse Engineering Project")
     (date "2023-03-14")
     (rev "DEV")
