File: schematic/right_angle/right_angle.kicad_pcb (KiCad board)
At the start: 2 copper layers, 82.5 x 20.3 mm, 3 parts, among them J12 Cartridge Port, J13 Cartridge Connector

Commit message: update with last few changes and fixes
Changed lines of the file:
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@@
     (property "ki_keywords" "connector")
     (attr through_hole)
-    (fp_text reference "J12" (at -18.6588 9.791) (layer "F.SilkS")
+    (fp_text reference "J12" (at -50.4952 2.5146) (layer "F.SilkS")
         (effects (font (size 1.27 1.27) (thickness 0.254)))
     )
@@
     (property "ki_keywords" "connector")
     (attr exclude_from_pos_files)
-    (fp_text reference "J13" (at 22.5958 -9.1814) (layer "F.SilkS")
+    (fp_text reference "J13" (at 43.4848 -5.9944) (layer "F.SilkS")
         (effects (font (size 1 1) (thickness 0.15)))
     )
@@
         (effects (font (size 1 1) (thickness 0.15)))
     )
-    (fp_line (start 1.524 2.54) (end 1.524 -4.572)
+    (fp_rect (start 1.524 -6.858) (end 41.656 3.302)
+      (stroke (width 0.1) (type solid)) (fill solid) (layer "B.Mask"))
+    (fp_rect (start 1.524 -6.858) (end 41.656 3.302)
+      (stroke (width 0.1) (type solid)) (fill solid) (layer "F.Mask"))
+    (fp_line (start 1.524 2.54) (end 1.524 -6.858)
       (stroke (width 0.1) (type solid)) (layer "Edge.Cuts"))
     (fp_line (start 2.032 3.302) (end 1.524 2.54)
@@
     (fp_line (start 41.148 3.302) (end 2.032 3.302)
       (stroke (width 0.1) (type solid)) (layer "Edge.Cuts"))
-    (fp_line (start 41.656 -4.572) (end 41.656 2.54)
+    (fp_line (start 41.656 -6.858) (end 41.656 2.54)
       (stroke (width 0.1) (type solid)) (layer "Edge.Cuts"))
     (fp_line (start 41.656 2.54) (end 41.148 3.302)
